Commit message: updated urdf for MoveIt!

File: ur_description/urdf/ur5.urdf (original).xacro (robot description, xacro)
@@ -311,48 +311,4 @@
       <child link="${prefix}tool0"/>
     </joint>
-    <!-- Begin: Custom environment elements -->
-    	<material name="transparent">
-		<color rgba="0 0 0 0.4"/>
-	</material>
-    <link name="room_link">
-      <visual>
-        <geometry>
-          <box size="0.7 2 1.5"/>
-        </geometry>
-        <origin xyz="0.36 0 0.75" rpy="0 0 0"/>
-        <material name="transparent"/>
-        <!--0.345/0.347-->
-      </visual>
-    </link>
-    <link name="robo_mount">
-      <visual>
-        <geometry>
-          <box size="0.08 0.15 0.15"/>
-        </geometry>
-        <origin xyz="0 0 0" rpy="0 0 0"/>
-      </visual>
-      <collision>
-        <geometry>
-          <box size="0.07 0.07 0.07"/>
-        </geometry>
-      </collision>
-    </link>
-    <link name="world" />
-    <joint name="world_joint" type="fixed">
-      <parent link="world" />
-      <child link = "room_link" />
-      <origin xyz="0.0 0.0 0.0" rpy="0.0 0.0 0.0" />
-    </joint>
-    <joint name="mount_platform_to_room" type="fixed">
-      <parent link="room_link" />
-      <child link = "robo_mount" />
-      <origin xyz="0.04 0.0 1.3" rpy="0.0 0.0 0.0" />
-    </joint>
-    <joint name="mount_platform_to_robot" type="fixed">
-      <parent link= "robo_mount" />
-      <child link = "base_link" />
-      <origin xyz="0.04 0 0" rpy="0 1.57 0" />
-    </joint>
-    <!-- End: Custom environment elements -->
   </xacro:macro>
 </robot>

File: ur_description/urdf/ur5_robot.urdf.xacro (robot description, xacro)
@@ -7,31 +7,6 @@
   <xacro:include filename="$(find ur_description)/urdf/ur5.urdf.xacro" />
   <!-- Barret Hand -->
-  <xacro:include filename="$(find barrett_hand_description)/urdf/bh280.urdf.xacro" ns="gripper" />
+  <xacro:include filename="$(find barrett_hand_description)/urdf/bh280.urdf.xacro" />
   <!-- arm -->
   <xacro:ur5_robot prefix="" joint_limited="false"/>
-  <link name="room_link">
-    <visual>
-      <geometry>
-        <box size="0 2 1.5"/>
-        <!-- <box size="0.7 2 1.5"/> -->
-      </geometry>
-      <origin xyz="0 0 0.75" rpy="0 0 0"/>
-    </visual>
-    <collision>
-      <geometry>
-        <box size="0 2 1.5"/>
-      </geometry>
-    </collision>
-  </link>
-  <link name="world" />
-  <joint name="world_joint" type="fixed">
-    <parent link="world" />
-    <child link = "room_link" />
-    <origin xyz="0.0 0.0 0.0" rpy="0.0 0.0 0.0" />
-  </joint>
-  <joint name="room_to_robot" type="fixed">
-    <parent link= "room_link" />
-    <child link = "base_link" />
-    <origin xyz="0.0 0 1.3" rpy="0 1.57 0" />
-  </joint>
 </robot>
